Commit message: Move Base Flex implementation.

File: bbblue_bot_description/urdf/bbblue_robot.xacro (robot description, xacro)
@@ -4,9 +4,9 @@
   <xacro:include filename="$(find bbblue_bot_description)/urdf/bbblue_robot_def.xacro" />
   <xacro:include filename="$(find bbblue_bot_description)/urdf/bbblue_robot_material.xacro" />
+  <xacro:include filename="$(find bbblue_bot_description)/urdf/bbblue_robot_wheels.xacro" />
   <!-- bbblue robot gazebo -->
   <xacro:include filename="$(find bbblue_bot_description)/urdf/bbblue_robot.gazebo" />
-  <xacro:include filename="$(find bbblue_bot_description)/urdf/bbblue_robot_wheels.xacro" />
   <!-- Base link -->
-  <link name="base_footprint">
+  <link name="base_link">
     <!-- visual>
         <origin xyz="0 0 0" rpy="0 0 0" />
@@ -19,5 +19,5 @@
   <joint name="base_footprint_joint" type="fixed">
     <origin xyz="0 0 ${2*casterRadius + chassisHeight}" rpy="0 0 0" />
-    <parent link="base_footprint"/>
+    <parent link="base_link"/>
     <child link="chassis" />
   </joint>
@@ -51,45 +51,12 @@
         z="${chassisHeight}"/>
     </inertial>
-    <visual>
-      <origin xyz="${casterOffsetX} 0 0"
-          rpy="0 0 0"/>
-      <geometry>
-        <mesh filename="package://bbblue_bot_description/meshes/caster_wheel.dae" />
-      </geometry>
-      <material name="grey" />
-    </visual>
-    <inertial>
-      <origin xyz="${casterOffsetX} 0 0"
-          rpy="0 0 0"/>
-      <mass value="${casterMass}"/>
-      <xacro:sphere_inertia
-        m="${casterMass}"
-        r="${casterRadius}"/>
-    </inertial>
-    <collision>
-      <origin xyz="${casterOffsetX} 0 0"
-          rpy="0 0 0"/>
-      <geometry>
-        <mesh filename="package://bbblue_bot_description/meshes/caster_wheel.dae" />
-      </geometry>
-      <surface>
-        <friction>
-          <ode>
-            <mu>0</mu>
-            <mu2>0</mu2>
-            <slip1>1.0</slip1>
-            <slip2>1.0</slip2>
-          </ode>
-        </friction>
-      </surface>
-    </collision>
   </link>
   <!-- Caster Joint -->
-  <!-- joint name="caster_joint" type="fixed">
+  <joint name="caster_joint" type="fixed">
     <parent link="chassis"/>
     <child link="caster_wheel"/>
-  </joint -->
+  </joint>
   <!-- Caster Wheel -->
-  <!-- link name="caster_wheel">
+  <link name="caster_wheel">
     <collision>
       <origin xyz="${casterOffsetX} 0 0"
@@ -125,8 +92,8 @@
         r="${casterRadius}"/>
     </inertial>
-  </link -->
+  </link>
   <!-- Wheel link -->
-  <xacro:wheel lr="left" tY="-1"/>
-  <xacro:wheel lr="right" tY="1"/>
+  <wheel lr="left" tY="-1" parent="chassis"/>
+  <wheel lr="right" tY="1" parent="chassis"/>
   <!-- Sensor models -->
   <xacro:include filename="$(find bbblue_bot_description)/urdf/bbblue_robot_sensors.xacro" />

File: bbblue_bot_description/urdf/bbblue_robot_def.xacro (robot description, xacro)
@@ -25,3 +25,4 @@
 	<xacro:property name="sonarOffsetX" value="0.066"/>
 	<!-- xacro:property name="sonarOffsetZ" value="0.0496"/ -->
+	<xacro:property name="x_reference_heading" value="90.0" />
 </robot>

File: bbblue_bot_description/urdf/bbblue_robot_sensors.xacro (robot description, xacro)
@@ -3,13 +3,13 @@
   <!-- Robot constants and properties -->
   <xacro:include filename="$(find bbblue_bot_description)/urdf/bbblue_robot_def.xacro" />
-  <!-- link name="sonar_link" -->
-  <joint name="sonar_link" type="fixed">
+  <!-- link name="laser_link" -->
+  <joint name="laser_joint" type="fixed">
     <axis xyz="0 1 0" />
-    <origin xyz="${sonarOffsetX} 0 -${(casterRadius / 2)}"
-            rpy="0 0 0"/>
+    <origin xyz="${sonarOffsetX} 0 ${(casterRadius / 2)}"
+            rpy="3.1415927 0 0"/>
     <parent link="chassis"/>
-    <child link="sonar_link"/>
+    <child link="laser_link"/>
   </joint>
-  <link name="sonar_link">
+  <link name="laser_link">
     <collision>
       <origin xyz="0 0 0"
@@ -34,5 +34,5 @@
       <origin xyz="0 0 0"
               rpy="0 0 0"/>
-      <xacro:box_inertia
+      <box_inertia
         m="${sonarMass}"
         x="${sonarLength}"

File: bbblue_bot_description/urdf/bbblue_robot_wheels.xacro (robot description, xacro)
@@ -34,5 +34,5 @@
     />
   </xacro:macro>
-  <xacro:macro name="wheel" params="lr tY">
+  <xacro:macro name="wheel" params="lr tY parent">
     <link name="${lr}_wheel">
       <collision>
@@ -56,5 +56,5 @@
         		rpy="${-tY*PI/2} 0 0" />
         <mass value="${wheelMass}"/>
-        <xacro:cylinder_inertia
+        <cylinder_inertia
           m="${wheelMass}"
           r="${wheelRadius}"
@@ -63,16 +63,22 @@
     </link>
     <gazebo reference="${lr}_wheel">
-      <mu1 value="1.0"/>
-      <mu2 value="1.0"/>
+      <mu1 value="10.0"/>
+      <mu2 value="10.0"/>
       <kp  value="10000000.0" />
       <kd>100.0</kd>
-      <minDepth>0.001</minDepth>
+      <minDepth>0.00</minDepth>
       <maxVel>1.0</maxVel>
-      <!--kd  value="1.0" />
-      <fdir1 value="1 0 0"/-->
+      <!-- kp>1000000.0</kp>
+      <kd>100.0</kd>
+      <mu1>200.0</mu1>
+      <mu2>100.0</mu2>
+      <fdir1>1 0 0</fdir1>
+      <maxVel>1.0</maxVel>
+      <minDepth>0.00</minDepth>
+      <implicitSpringDamper>1</implicitSpringDamper -->
       <material>Gazebo/FlatBlack</material>
     </gazebo>
     <joint name="${lr}_wheel_hinge" type="continuous">
-      <parent link="chassis"/>
+      <parent link="${parent}"/>
       <child link="${lr}_wheel"/>
       <origin
@@ -82,19 +88,17 @@
       		  rpy="0 0 0" />
       <!--limit effort="100" velocity="10"/-->
-      <limit effort="0.0" velocity="0.0"/>
+      <limit effort="100" velocity="10"/>
       <joint_properties damping="0.0" friction="0.0"/>
     </joint>
-<!--
-  http://gazebosim.org/tutorials/?tut=ros_control
--->
-    <transmission name="${lr}_trans">
+    <transmission name="${lr}_joint_trans">
       <type>transmission_interface/SimpleTransmission</type>
       <joint name="${lr}_wheel_hinge">
-        <hardwareInterface>hardware_interface/EffortJointInterface</hardwareInterface>
+        <hardwareInterface>hardware_interface/VelocityJointInterface</hardwareInterface>
+        <!-- hardwareInterface>hardware_interface/EffortJointInterface</hardwareInterface -->
       </joint>
-      <actuator name="${lr}Motor">
-        <hardwareInterface>hardware_interface/EffortJointInterface</hardwareInterface>
-        <mechanicalReduction>10</mechanicalReduction>
-        <!--mechanicalReduction>1</mechanicalReduction-->
+      <actuator name="${lr}_joint_motor">
+        <hardwareInterface>hardware_interface/VelocityJointInterface</hardwareInterface>
+        <!-- hardwareInterface>hardware_interface/EffortJointInterface</hardwareInterface -->
+        <mechanicalReduction>1</mechanicalReduction>
       </actuator>
     </transmission>
